Commit message: make more flexible

File: ranger_mini/ranger_mini_v2/urdf/ranger_mini.xacro (robot description, xacro)
@@ -1,266 +1,5 @@
-<?xml version="1.0"?>
-<robot name="ranger_mini_v2"
-    xmlns:xacro="http://ros.org/wiki/xacro">
-    <xacro:include filename="$(find ranger_mini_v2)/urdf/ranger_l.xacro" />
-    <xacro:include filename="$(find ranger_mini_v2)/urdf/ranger_r.xacro" />
-    <!-- Variables -->
-    <xacro:property name="M_PI" value="3.14159"/>
-    <!-- Vehicle Geometries -->
-    <xacro:property name="base_x_size" value="1.0" />
-    <xacro:property name="base_y_size" value="0.380000" />
-    <xacro:property name="base_z_size" value="0.210000" />
-    <xacro:property name="wheelbase" value="0.498" />
-    <xacro:property name="track" value="0.58306" />
-    <xacro:property name="wheel_vertical_offset" value="-0.0702" />
-    <xacro:property name="wheel_length" value="1.1653e-01" />
-    <xacro:property name="wheel_radius" value="1.6459e-01" />
-    <!-- Base link -->
-    <link name="base_link">
-        <visual>
-            <origin xyz="0 0 0" rpy="1.57 0 3.14 " />
-            <geometry>
-                <mesh filename="package://ranger_mini_v2/meshes/ranger_base.dae" />
-            </geometry>
-        </visual>
-        <collision>
-            <origin xyz="0 0 0.008" rpy="0 0 0" />
-            <geometry>
-                <box size="1 1 1"/>
-            </geometry>
-        </collision>
-        <collision>
-            <origin xyz="0 0 0" rpy="0 0 0" />
-            <geometry>
-                <box size="1 1 1"/>
-            </geometry>
-        </collision>
-    </link>
-   <link name="fl_steering_wheel_link">
-        <visual>
-            <origin xyz="0 0 0" rpy="1.57 0 3.14 " />
-            <geometry>
-                <cylinder radius="0.001" length="0.001"/>
-            </geometry>
-        </visual>
-        <collision>
-            <origin xyz="0 0 0.008" rpy="0 0 0" />
-            <geometry>
-                <box size="1 1 1"/>
-            </geometry>
-        </collision>
-        <collision>
-            <origin xyz="0 0 0" rpy="0 0 0" />
-            <geometry>
-                <cylinder radius="0.001" length="0.001"/>
-            </geometry>
-        </collision>
-    </link>
-    <joint name="fl_steering_wheel" type="revolute">
-        <origin xyz="0.23 0.206 -0.1" rpy="0 0 0" />
-        <parent link="base_link"/>
-        <child link="fl_steering_wheel_link"/>
-        <axis xyz="0 0 1" rpy="0 0 0" />
-        <limit effort="5" velocity="6.28"  lower="-2.1" upper="2.1" />
-    </joint>
-        <link name="fl_wheel_link">
-            <inertial>
-                <mass value="8" />
-                <origin xyz="0 0 0" />
-                <inertia ixx="0.1171" ixy="0" ixz="0" iyy="0.1361" iyz="0" izz="0.1171" />
-            </inertial>
-            <visual>
-                <origin xyz="0.23 -0.2 0.1" rpy="1.57 0 0" />
-                <geometry>
-                    <mesh filename="package://ranger_mini_v2/meshes/fr.dae" />
-                </geometry>
-            </visual>
-            <collision>
-                <origin xyz="0 0 0" rpy="0 0 0" />
-                <geometry>
-                    <cylinder length="0.1" radius="0.1" />
-                </geometry>
-                     <contact>
-                         <ode>
-                        <min_depth>0.001</min_depth>
-                         </ode>
-                    </contact>
-            </collision>
-        </link>
-        <joint name="fl_wheel" type="continuous">
-            <origin xyz="0.0 0.0 0.0" rpy="0 0 0" />
-            <parent link="fl_steering_wheel_link"/>
-            <child link="fl_wheel_link"/>
-            <axis xyz="0 0 1" rpy="0 0 0" />
-        </joint>
-   <link name="fr_steering_wheel_link">
-        <visual>
-            <origin xyz="0 0 0" rpy="1.57 0 3.14 " />
-            <geometry>
-                <cylinder radius="0.001" length="0.001"/>
-            </geometry>
-        </visual>
-        <collision>
-            <origin xyz="0 0 0.008" rpy="0 0 0" />
-            <geometry>
-                <box size="1 1 1"/>
-            </geometry>
-        </collision>
-        <collision>
-            <origin xyz="0 0 0" rpy="0 0 0" />
-            <geometry>
-                <cylinder radius="0.001" length="0.001"/>
-            </geometry>
-        </collision>
-    </link>
-    <joint name="fr_steering_wheel" type="revolute">
-        <origin xyz="0.23 -0.206 -0.1" rpy="0 0 0" />
-        <parent link="base_link"/>
-        <child link="fr_steering_wheel_link"/>
-        <axis xyz="0 0 1" rpy="0 0 0" />
-        <limit effort="5" velocity="6.28"  lower="-2.1" upper="2.1" />
-    </joint>
-        <link name="fr_wheel_link">
-            <inertial>
-                <mass value="8" />
-                <origin xyz="0 0 0" />
-                <inertia ixx="0.1171" ixy="0" ixz="0" iyy="0.1361" iyz="0" izz="0.1171" />
-            </inertial>
-            <visual>
-                <origin xyz="0.23 0.2 0.1" rpy="1.57 0 0" />
-                <geometry>
-                    <mesh filename="package://ranger_mini_v2/meshes/fl.dae" />
-                </geometry>
-            </visual>
-            <collision>
-                <origin xyz="0 0 0" rpy="0 0 0" />
-                <geometry>
-                    <cylinder length="0.1" radius="0.1" />
-                </geometry>
-                     <contact>
-                         <ode>
-                        <min_depth>0.001</min_depth>
-                         </ode>
-                    </contact>
-            </collision>
-        </link>
-        <joint name="fr_wheel" type="continuous">
-            <origin xyz="0.0 0.0 0.0" rpy="0 0 0" />
-            <parent link="fr_steering_wheel_link"/>
-            <child link="fr_wheel_link"/>
-            <axis xyz="0 0 1" rpy="0 0 0" />
-        </joint>
-   <link name="rl_steering_wheel_link">
-        <visual>
-            <origin xyz="0 0 0" rpy="1.57 0 3.14 " />
-            <geometry>
-                <cylinder radius="0.001" length="0.001"/>
-            </geometry>
-        </visual>
-        <collision>
-            <origin xyz="0 0 0.008" rpy="0 0 0" />
-            <geometry>
-                <box size="1 1 1"/>
-            </geometry>
-        </collision>
-        <collision>
-            <origin xyz="0 0 0" rpy="0 0 0" />
-            <geometry>
-                <cylinder radius="0.001" length="0.001"/>
-            </geometry>
-        </collision>
-    </link>
-    <joint name="rl_steering_wheel" type="revolute">
-        <origin xyz="-0.23 0.206 -0.1" rpy="0 0 0" />
-        <parent link="base_link"/>
-        <child link="rl_steering_wheel_link"/>
-        <axis xyz="0 0 1" rpy="0 0 0" />
-        <limit effort="5" velocity="6.28"  lower="-2.1" upper="2.1" />
-    </joint>
-        <link name="rl_wheel_link">
-            <inertial>
-                <mass value="8" />
-                <origin xyz="0 0 0" />
-                <inertia ixx="0.1171" ixy="0" ixz="0" iyy="0.1361" iyz="0" izz="0.1171" />
-            </inertial>
-            <visual>
-                <origin xyz="0.23 -0.2 0.1" rpy="1.57 0 0" />
-                <geometry>
-                    <mesh filename="package://ranger_mini_v2/meshes/fr.dae" />
-                </geometry>
-            </visual>
-            <collision>
-                <origin xyz="0 0 0" rpy="0 0 0" />
-                <geometry>
-                    <cylinder length="0.1" radius="0.1" />
-                </geometry>
-                     <contact>
-                         <ode>
-                        <min_depth>0.001</min_depth>
-                         </ode>
-                    </contact>
-            </collision>
-        </link>
-        <joint name="rl_wheel" type="continuous">
-            <origin xyz="0.0 0.0 0.0 " rpy="0 0 0" />
-            <parent link="rl_steering_wheel_link"/>
-            <child link="rl_wheel_link"/>
-            <axis xyz="0 0 1" rpy="0 0 0" />
-        </joint>
-   <link name="rr_steering_wheel_link">
-        <visual>
-            <origin xyz="0 0 0" rpy="1.57 0 3.14 " />
-            <geometry>
-                <cylinder radius="0.001" length="0.001"/>
-            </geometry>
-        </visual>
-        <collision>
-            <origin xyz="0 0 0.008" rpy="0 0 0" />
-            <geometry>
-                <box size="1 1 1"/>
-            </geometry>
-        </collision>
-        <collision>
-            <origin xyz="0 0 0" rpy="0 0 0" />
-            <geometry>
-                <cylinder radius="0.001" length="0.001"/>
-            </geometry>
-        </collision>
-    </link>
-    <joint name="rr_steering_wheel" type="revolute">
-        <origin xyz="-0.23 -0.206 -0.1" rpy="0 0 0" />
-        <parent link="base_link"/>
-        <child link="rr_steering_wheel_link"/>
-        <axis xyz="0 0 1" rpy="0 0 0" />
-        <limit effort="5" velocity="6.28"  lower="-2.1" upper="2.1" />
-    </joint>
-        <link name="rr_wheel_link">
-            <inertial>
-                <mass value="8" />
-                <origin xyz="0 0 0" />
-                <inertia ixx="0.1171" ixy="0" ixz="0" iyy="0.1361" iyz="0" izz="0.1171" />
-            </inertial>
-            <visual>
-                <origin xyz="0.23 0.2 0.1" rpy="1.57 0 0" />
-                <geometry>
-                    <mesh filename="package://ranger_mini_v2/meshes/fl.dae" />
-                </geometry>
-            </visual>
-            <collision>
-                <origin xyz="0 0 0" rpy="0 0 0" />
-                <geometry>
-                    <cylinder length="0.1" radius="0.1" />
-                </geometry>
-                     <contact>
-                         <ode>
-                        <min_depth>0.001</min_depth>
-                         </ode>
-                    </contact>
-            </collision>
-        </link>
-        <joint name="rr_wheel" type="continuous">
-            <origin xyz="0.0 0.0 0.0 " rpy="0 0 0" />
-            <parent link="rr_steering_wheel_link"/>
-            <child link="rr_wheel_link"/>
-            <axis xyz="0 0 1" rpy="0 0 0" />
-        </joint>
+<?xml version="1.0" ?>
+<robot name="ranger_mini_v2" xmlns:xacro="http://www.ros.org/wiki/xacro">
+  <xacro:include filename="$(find ranger_mini_v2)/urdf/ranger_mini_macro.xacro"/>
+  <xacro:ranger_mini_v2 attach_to_world="yes"/>
 </robot>
