Commit message: add simplified base

File: ranger_mini/ranger_mini_v2/urdf/ranger_mini_macro.xacro (robot description, xacro)
@@ -30,5 +30,5 @@
             <origin xyz="0 0 0" rpy="1.57 0 3.14 " />
             <geometry>
-                <mesh filename="package://ranger_mini_v2/meshes/ranger_base.dae" />
+                <mesh filename="package://ranger_mini_v2/meshes/ranger_base_simplified.dae" />
             </geometry>
         </visual>

Commit message: remove insane collision geometry

File: ranger_mini/ranger_mini_v2/urdf/ranger_mini_macro.xacro (robot description, xacro)
@@ -33,16 +33,16 @@
             </geometry>
         </visual>
-        <collision>
-            <origin xyz="0 0 0.008" rpy="0 0 0" />
-            <geometry>
-                <box size="1 1 1"/>
-            </geometry>
-        </collision>
-        <collision>
-            <origin xyz="0 0 0" rpy="0 0 0" />
-            <geometry>
-                <box size="1 1 1"/>
-            </geometry>
-        </collision>
+        <!-- <collision>
+            <origin xyz="0 0 0.008" rpy="0 0 0" />
+            <geometry>
+                <box size="1 1 1"/>
+            </geometry>
+        </collision>
+        <collision>
+            <origin xyz="0 0 0" rpy="0 0 0" />
+            <geometry>
+                <box size="1 1 1"/>
+            </geometry>
+        </collision> -->
     </link>
    <link name="fl_steering_wheel_link">
@@ -53,16 +53,16 @@
             </geometry>
         </visual>
-        <collision>
-            <origin xyz="0 0 0.008" rpy="0 0 0" />
-            <geometry>
-                <box size="1 1 1"/>
-            </geometry>
-        </collision>
-        <collision>
-            <origin xyz="0 0 0" rpy="0 0 0" />
-            <geometry>
-                <cylinder radius="0.001" length="0.001"/>
-            </geometry>
-        </collision>
+        <!-- <collision>
+            <origin xyz="0 0 0.008" rpy="0 0 0" />
+            <geometry>
+                <box size="1 1 1"/>
+            </geometry>
+        </collision>
+        <collision>
+            <origin xyz="0 0 0" rpy="0 0 0" />
+            <geometry>
+                <cylinder radius="0.001" length="0.001"/>
+            </geometry>
+        </collision> -->
     </link>
     <joint name="fl_steering_wheel" type="revolute">
@@ -110,16 +110,16 @@
             </geometry>
         </visual>
-        <collision>
-            <origin xyz="0 0 0.008" rpy="0 0 0" />
-            <geometry>
-                <box size="1 1 1"/>
-            </geometry>
-        </collision>
-        <collision>
-            <origin xyz="0 0 0" rpy="0 0 0" />
-            <geometry>
-                <cylinder radius="0.001" length="0.001"/>
-            </geometry>
-        </collision>
+        <!-- <collision>
+            <origin xyz="0 0 0.008" rpy="0 0 0" />
+            <geometry>
+                <box size="1 1 1"/>
+            </geometry>
+        </collision>
+        <collision>
+            <origin xyz="0 0 0" rpy="0 0 0" />
+            <geometry>
+                <cylinder radius="0.001" length="0.001"/>
+            </geometry>
+        </collision> -->
     </link>
     <joint name="fr_steering_wheel" type="revolute">
@@ -167,16 +167,16 @@
             </geometry>
         </visual>
-        <collision>
-            <origin xyz="0 0 0.008" rpy="0 0 0" />
-            <geometry>
-                <box size="1 1 1"/>
-            </geometry>
-        </collision>
-        <collision>
-            <origin xyz="0 0 0" rpy="0 0 0" />
-            <geometry>
-                <cylinder radius="0.001" length="0.001"/>
-            </geometry>
-        </collision>
+        <!-- <collision>
+            <origin xyz="0 0 0.008" rpy="0 0 0" />
+            <geometry>
+                <box size="1 1 1"/>
+            </geometry>
+        </collision>
+        <collision>
+            <origin xyz="0 0 0" rpy="0 0 0" />
+            <geometry>
+                <cylinder radius="0.001" length="0.001"/>
+            </geometry>
+        </collision> -->
     </link>
     <joint name="rl_steering_wheel" type="revolute">
@@ -224,16 +224,16 @@
             </geometry>
         </visual>
-        <collision>
-            <origin xyz="0 0 0.008" rpy="0 0 0" />
-            <geometry>
-                <box size="1 1 1"/>
-            </geometry>
-        </collision>
-        <collision>
-            <origin xyz="0 0 0" rpy="0 0 0" />
-            <geometry>
-                <cylinder radius="0.001" length="0.001"/>
-            </geometry>
-        </collision>
+        <!-- <collision>
+            <origin xyz="0 0 0.008" rpy="0 0 0" />
+            <geometry>
+                <box size="1 1 1"/>
+            </geometry>
+        </collision>
+        <collision>
+            <origin xyz="0 0 0" rpy="0 0 0" />
+            <geometry>
+                <cylinder radius="0.001" length="0.001"/>
+            </geometry>
+        </collision> -->
     </link>
     <joint name="rr_steering_wheel" type="revolute">

Commit message: temp remove things before moving package to extend_ranger

File: ranger_mini/ranger_mini_v2/urdf/ranger_mini_macro.xacro (robot description, xacro)
@@ -30,5 +30,5 @@
             <origin xyz="0 0 0" rpy="1.57 0 3.14 " />
             <geometry>
-                <mesh filename="package://ranger_mini_v2/meshes/ranger_base_simplified.dae" />
+                <mesh filename="package://ranger_mini_v2/meshes/ranger_base.dae" />
             </geometry>
         </visual>
